Commit message: Solved errors with inertia
Signed-off-by: Juancams <jc.manzanares.serrano@gmail.com>

File: urdf/base_camera.urdf.xacro (robot description, xacro)
@@ -4,9 +4,4 @@
   <xacro:macro name="base" params="camera_frame">
     <link name="base_oak">
-      <inertial>
-        <mass value="1.0"/>
-        <origin xyz="0 0 0" rpy="1.56 0.00291 -1.56"/>
-        <inertia ixx="0.1" ixy="0.0" ixz="0.0" iyy="0.1" iyz="0.0" izz="0.1"/>
-      </inertial>
       <visual>
         <origin xyz="0 0 0" rpy="1.56 0 -1.56"/>
@@ -19,5 +14,5 @@
       </visual>
       <collision>
-        <origin xyz="0 0 0" rpy="1.56  -1.56"/>
+        <origin xyz="0 0 0" rpy="1.56 0 -1.56"/>
         <geometry>
           <mesh filename="package://oak_d_camera/meshes/oak_dlite_base.stl" scale="0.001 0.001 0.001"/>
@@ -32,5 +27,7 @@
     <link name="base_footprint">
         <inertial>
+        <mass value="0.0"/>
         <origin xyz="0 0 0" rpy="0 0 0"/>
+        <inertia ixx="0.0" ixy="0.0" ixz="0.0" iyy="0.0" iyz="0.0" izz="0.0"/>
       </inertial>
     </link>

Commit message: Changes to make xyz rpy parameters work
Signed-off-by: Juancams <jc.manzanares.serrano@gmail.com>

File: urdf/base_camera.urdf.xacro (robot description, xacro)
@@ -2,5 +2,5 @@
 <robot xmlns:xacro="http://www.ros.org/wiki/xacro" name="base_oak">
   <!-- Macro base -->
-  <xacro:macro name="base" params="camera_frame">
+  <xacro:macro name="base" params="camera_frame cam_pos_x cam_pos_y cam_pos_z cam_roll cam_pitch cam_yaw">
     <link name="base_oak">
       <visual>
@@ -35,5 +35,5 @@
       <parent link="base_footprint"/>
       <child link="${camera_frame}"/>
-      <origin xyz="0 0 0.08863" rpy="0 -0.0508 0"/>
+      <origin xyz="${cam_pos_x} ${cam_pos_y} ${cam_pos_z + 0.08863}" rpy="${cam_roll} ${- 0.0508 - cam_pitch} ${cam_yaw}"/>
     </joint>
     <link name="${camera_frame}" />

File: urdf/base_descr.urdf.xacro (robot description, xacro)
@@ -13,11 +13,13 @@
 	<xacro:arg name="rs_compat" default="false" />
     <xacro:arg name="use_base" default="false" />
-	<xacro:include filename="$(find depthai_descriptions)/urdf/include/depthai_macro.urdf.xacro" />
+	<xacro:include filename="$(find oak_d_camera)/urdf/include/depthai_macro.urdf.xacro" />
     <xacro:include filename="$(find oak_d_camera)/urdf/base_camera.urdf.xacro" />
     <xacro:if value="$(arg use_base)">
-        <xacro:base camera_frame="$(arg parent_frame)" />
+        <xacro:base camera_frame="$(arg parent_frame)" cam_pos_x="$(arg cam_pos_x)" cam_pos_y="$(arg cam_pos_y)" cam_pos_z="$(arg cam_pos_z)" cam_roll="$(arg cam_roll)" cam_pitch="$(arg cam_pitch)" cam_yaw="$(arg cam_yaw)" />
     </xacro:if>
     <xacro:unless value="$(arg use_base)">
-        <link name="$(arg parent_frame)" />
+        <link name="$(arg parent_frame)" >
+			<pose xyz="$(arg cam_pos_x) $(arg cam_pos_y) $(arg cam_pos_z)" rpy="$(arg cam_roll) $(arg cam_pitch) $(arg cam_yaw)" />
+		</link>
     </xacro:unless>
 	<xacro:depthai_camera camera_name="$(arg camera_name)" parent="$(arg parent_frame)"

Commit message: new calibration parameters
Signed-off-by: Jose Miguel <josemiguel.guerrero@urjc.es>

File: urdf/base_camera.urdf.xacro (robot description, xacro)
@@ -35,5 +35,5 @@
       <parent link="base_footprint"/>
       <child link="${camera_frame}"/>
-      <origin xyz="${cam_pos_x} ${cam_pos_y} ${cam_pos_z + 0.08863}" rpy="${cam_roll} ${- 0.0508 - cam_pitch} ${cam_yaw}"/>
+      <origin xyz="${cam_pos_x} ${cam_pos_y} ${cam_pos_z + 0.08863}" rpy="${cam_roll} ${- 0.0858 - cam_pitch} ${cam_yaw}"/>
     </joint>
     <link name="${camera_frame}" />
