Commit message: Adding IMU
Signed-off-by: Jose Miguel <josemiguel.guerrero@urjc.es>

File: urdf/include/base_macro.urdf.xacro (robot description, xacro)
@@ -69,4 +69,12 @@
 			<xacro:property name="imu_y" value="0.0" />
 		</xacro:if>
+		<xacro:if value="${model == 'OAK-D-LITE'}">
+			<xacro:property name="imu_offset_x" value="0.0" />
+			<xacro:property name="imu_offset_y" value="-0.015" />
+			<xacro:property name="imu_offset_z" value="-0.013662" />
+			<xacro:property name="imu_r" value="0.0" />
+			<xacro:property name="imu_p" value="${M_PI/2.0}" />
+			<xacro:property name="imu_y" value="0.0" />
+		</xacro:if>
 		<xacro:if value="${model == 'OAK-D-PRO'}">
 			<xacro:property name="imu_offset_x" value="-0.008" />

File: urdf/include/depthai_macro.urdf.xacro (robot description, xacro)
@@ -28,5 +28,5 @@
 			<xacro:property name="baseline" value="0.02" />
 		</xacro:if>
-		<xacro:if value="${model in ['OAK-D', 'OAK-D-PRO', 'OAK-D-POE']}">
+		<xacro:if value="${model in ['OAK-D', 'OAK-D-LITE', 'OAK-D-PRO', 'OAK-D-POE']}">
 			<xacro:property name="has_imu" value="true" />
 		</xacro:if>
